File: PCIe.kicad_sch (KiCad schematic)
At the start: 24 parts, among them J11 10018783-11200TLF, U8 AP64501SP-13

Commit message: pulled in bitcrane fan and data connectors and edge cuts. most placement done. started routing
Parts:
- removed C23, C24, C25, C26, C27, C28: 10u 35v, Capacitor_SMD:C_0805_2012Metric, symbol Device:C
- removed C29, C30: 0.1uF, Capacitor_SMD:C_0402_1005Metric, symbol Device:C
- removed C31, C33: nf, Capacitor_SMD:C_0402_1005Metric, symbol Device:C
- removed C32: 1.2nF, Capacitor_SMD:C_0402_1005Metric, symbol Device:C
- removed C34, C35, C36, C37: 10u, Capacitor_SMD:C_0805_2012Metric, symbol Device:C
- removed C38: 100uF, Capacitor_Tantalum_SMD:CP_EIA-7343-31_Kemet-D, symbol Device:CP
- removed J11: 10018783-11200TLF, CM4IO:PCIex1-36, symbol CM4IO:PCIe-x1
- removed L1: SRN6045TA-3R3Y, Inductor_SMD:L_Bourns_SRN6045TA, symbol pspice:INDUCTOR
- removed R19: 10R, Resistor_SMD:R_0402_1005Metric, symbol Device:R_US
- removed R20: 12K 1%, Resistor_SMD:R_0402_1005Metric, symbol Device:R_US
- removed R21: 47K 1%, Resistor_SMD:R_0402_1005Metric, symbol Device:R_US
- removed R22: 15K 1%, Resistor_SMD:R_0402_1005Metric, symbol Device:R_US
- removed TP5: TestPoint, TestPoint:TestPoint_Pad_D1.5mm, symbol Connector:TestPoint
- removed U8: AP64501SP-13, Package_SO:SOIC-8-1EP_3.9x4.9mm_P1.27mm_EP2.95x4.9mm_Mask2.71x3.4mm_ThermalVias, symbol CM4IO:AP64351
Connections:
- no-connect marks 6 -> 0
Other:
- note removed: "3.3v @ 3.3A PSU for PCIe Only ( 12v Input )"
- note removed: "NB PCIe x1 takes a maximum of +12v @0.6A or +3.3v@3A , 10Watts combined"
- note removed: "PCIe x1 connector"
- note removed: "TX and RX have PN swaps to improve routing"
