File: CM4_GPIO.kicad_sch (KiCad schematic)
At the start: 17 parts, among them J10 Conn_02x03_Odd_Even, J8 Conn_01x02, J9 THD-20-R, U6 74LVC1G07SE-7, U7 MagJack-A70-112-331N126

Commit message: lots of routing. lots more to do
Parts:
- R17, R18: value 470R -> 470
Connections:
- net +3.3v renamed 3V3
- net +5v renamed 5V
- net GPIO9 renamed RXD4
Changed lines of the file:
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@@
     (effects (font (size 1.27 1.27)) (justify right bottom))
   )
-  (label "+3.3v" (at 33.02 115.57 180) (fields_autoplaced)
+  (label "3V3" (at 33.02 115.57 180) (fields_autoplaced)
     (effects (font (size 1.27 1.27)) (justify right bottom))
   )
@@
     (effects (font (size 1.27 1.27)) (justify right bottom))
   )
-  (label "+3.3v" (at 191.135 121.285 180) (fields_autoplaced)
+  (label "3V3" (at 191.135 121.285 180) (fields_autoplaced)
     (effects (font (size 1.27 1.27)) (justify right bottom))
   )
@@
     (effects (font (size 1.27 1.27)) (justify right bottom))
   )
-  (label "+5v" (at 170.18 24.13 180) (fields_autoplaced)
+  (label "5V" (at 170.18 24.13 180) (fields_autoplaced)
     (effects (font (size 1.27 1.27)) (justify right bottom))
   )
@@
     (effects (font (size 1.27 1.27)) (justify right bottom))
   )
-  (label "+3.3v" (at 148.59 24.13 180) (fields_autoplaced)
+  (label "3V3" (at 148.59 24.13 180) (fields_autoplaced)
     (effects (font (size 1.27 1.27)) (justify right bottom))
   )
@@
     (effects (font (size 1.27 1.27)) (justify left bottom))
   )
-  (label "+3.3v" (at 33.02 123.19 180) (fields_autoplaced)
+  (label "3V3" (at 33.02 123.19 180) (fields_autoplaced)
     (effects (font (size 1.27 1.27)) (justify right bottom))
   )
@@
     (effects (font (size 1.27 1.27)) (justify right bottom))
   )
-  (label "+5v" (at 106.68 115.57 180) (fields_autoplaced)
+  (label "5V" (at 106.68 115.57 180) (fields_autoplaced)
     (effects (font (size 1.27 1.27)) (justify right bottom))
   )
@@
     (effects (font (size 1.27 1.27)) (justify left bottom))
   )
-  (label "+3.3v" (at 116.84 17.78 180) (fields_autoplaced)
+  (label "3V3" (at 116.84 17.78 180) (fields_autoplaced)
     (effects (font (size 1.27 1.27)) (justify right bottom))
   )
@@
     (effects (font (size 1.27 1.27)) (justify left bottom))
   )
-  (label "+3.3v" (at 243.84 72.39 180) (fields_autoplaced)
+  (label "3V3" (at 243.84 72.39 180) (fields_autoplaced)
     (effects (font (size 1.27 1.27)) (justify right bottom))
   )
@@
     (effects (font (size 1.27 1.27)) (justify right bottom))
   )
-  (label "+3.3v" (at 179.705 137.795 180) (fields_autoplaced)
+  (label "3V3" (at 179.705 137.795 180) (fields_autoplaced)
     (effects (font (size 1.27 1.27)) (justify right bottom))
   )
@@
     )
   )
-  (hierarchical_label "+5v" (shape input) (at 114.3 115.57 0) (fields_autoplaced)
+  (hierarchical_label "5V" (shape input) (at 114.3 115.57 0) (fields_autoplaced)
     (effects (font (size 1.27 1.27)) (justify left))
   )
@@
     (effects (font (size 1.27 1.27)) (justify left))
   )
+  (hierarchical_label "RXD4" (shape input) (at 25.4 67.31 180) (fields_autoplaced)
+    (effects (font (size 1.27 1.27)) (justify right))
+  )
   (hierarchical_label "TXD5" (shape output) (at 114.3 57.15 0) (fields_autoplaced)
     (effects (font (size 1.27 1.27)) (justify left))
@@
     (effects (font (size 1.27 1.27)) (justify left))
   )
-  (hierarchical_label "+3.3v" (shape output) (at 25.4 123.19 180) (fields_autoplaced)
+  (hierarchical_label "3V3" (shape output) (at 25.4 123.19 180) (fields_autoplaced)
     (effects (font (size 1.27 1.27)) (justify right))
   )
@@
       (effects (font (size 1.27 1.27)))
     )
-    (property "Value" "470R" (at 232.41 71.9836 90)
+    (property "Value" "470" (at 232.41 71.9836 90)
       (effects (font (size 1.27 1.27)))
     )
@@
       (effects (font (size 1.27 1.27)))
     )
-    (property "Value" "470R" (at 232.41 82.55 90)
+    (property "Value" "470" (at 232.41 82.55 90)
       (effects (font (size 1.27 1.27)))
     )
