File: USB2-HUB.kicad_sch (KiCad schematic)
At the start: 31 parts, among them J1 USB_OTG, J2 690-008-221-904, U1 FSUSB42MUX, U2 USB2514B-I/M2, U3 TPD4EUSB30, U4 AP22653W6, Y1 24MHz

Commit message: lots of routing. lots more to do
Parts:
- R1, R2: value 2.2K 1% -> 2.2k 1%
- R3, R4, R5, R7: value 36K 1% -> 36k 1%
- R6: value 12K 1% -> 12k 1%
- R8: value 15K 1% -> 15k 1%
Connections:
- net +3.3v renamed 3V3
- net +5v renamed 5V
Changed lines of the file:
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@@
     (effects (font (size 1.27 1.27)) (justify left bottom))
   )
-  (label "+3.3v" (at 31.75 55.88 0) (fields_autoplaced)
+  (label "3V3" (at 31.75 55.88 0) (fields_autoplaced)
     (effects (font (size 1.27 1.27)) (justify left bottom))
   )
@@
     (effects (font (size 1.27 1.27)) (justify left bottom))
   )
-  (label "+3.3v" (at 68.58 165.1 0) (fields_autoplaced)
-    (effects (font (size 1.27 1.27)) (justify left bottom))
-  )
-  (label "+5v" (at 167.64 77.47 0) (fields_autoplaced)
+  (label "3V3" (at 68.58 165.1 0) (fields_autoplaced)
+    (effects (font (size 1.27 1.27)) (justify left bottom))
+  )
+  (label "5V" (at 167.64 77.47 0) (fields_autoplaced)
     (effects (font (size 1.27 1.27)) (justify left bottom))
   )
@@
     (effects (font (size 1.27 1.27)) (justify left bottom))
   )
-  (label "+3.3v" (at 107.95 73.66 0) (fields_autoplaced)
+  (label "3V3" (at 107.95 73.66 0) (fields_autoplaced)
     (effects (font (size 1.27 1.27)) (justify left bottom))
   )
@@
     (effects (font (size 1.27 1.27)) (justify right))
   )
-  (hierarchical_label "+3.3v" (shape input) (at 68.58 165.1 180) (fields_autoplaced)
+  (hierarchical_label "3V3" (shape input) (at 68.58 165.1 180) (fields_autoplaced)
     (effects (font (size 1.27 1.27)) (justify right))
   )
@@
     (effects (font (size 1.27 1.27)) (justify right))
   )
-  (hierarchical_label "+5v" (shape input) (at 167.64 77.47 180) (fields_autoplaced)
+  (hierarchical_label "5V" (shape input) (at 167.64 77.47 180) (fields_autoplaced)
     (effects (font (size 1.27 1.27)) (justify right))
   )
@@
       (effects (font (size 1.27 1.27)) (justify left))
     )
-    (property "Value" "2.2K 1%" (at 42.418 46.863 0)
+    (property "Value" "2.2k 1%" (at 42.418 46.863 0)
       (effects (font (size 1.27 1.27)) (justify left))
     )
@@
       (effects (font (size 1.27 1.27)) (justify left))
     )
-    (property "Value" "2.2K 1%" (at 23.495 73.66 0)
+    (property "Value" "2.2k 1%" (at 23.495 73.66 0)
       (effects (font (size 1.27 1.27)) (justify left))
     )
@@
       (effects (font (size 1.27 1.27)) (justify left))
     )
-    (property "Value" "36K 1%" (at 81.28 149.225 90)
+    (property "Value" "36k 1%" (at 81.28 149.225 90)
       (effects (font (size 1.27 1.27)) (justify left))
     )
@@
       (effects (font (size 1.27 1.27)) (justify left))
     )
-    (property "Value" "36K 1%" (at 73.66 149.225 90)
+    (property "Value" "36k 1%" (at 73.66 149.225 90)
       (effects (font (size 1.27 1.27)) (justify left))
     )
@@
       (effects (font (size 1.27 1.27)) (justify left))
     )
-    (property "Value" "36K 1%" (at 66.04 149.225 90)
+    (property "Value" "36k 1%" (at 66.04 149.225 90)
       (effects (font (size 1.27 1.27)) (justify left))
     )
@@
       (effects (font (size 1.27 1.27)) (justify left))
     )
-    (property "Value" "15K 1%" (at 222.25 76.2 90)
+    (property "Value" "15k 1%" (at 222.25 76.2 90)
       (effects (font (size 1.27 1.27)) (justify left))
     )
@@
       (effects (font (size 1.27 1.27)) (justify left))
     )
-    (property "Value" "12K 1%" (at 86.36 106.68 90)
+    (property "Value" "12k 1%" (at 86.36 106.68 90)
       (effects (font (size 1.27 1.27)) (justify left))
     )
@@
       (effects (font (size 1.27 1.27)) (justify left))
     )
-    (property "Value" "36K 1%" (at 88.9 149.225 90)
-      (effects (font (size 1.27 1.27)) (justify left))
-    )
+    (property "Value" "36k 1%" (at 88.9 149.225 90)
+      (effects (font (size 1.27 1.27)) (justify left))
+    )
