File: bitcart.kicad_sch (KiCad schematic)
At the start: 4 parts

Commit message: lots of routing. lots more to do
Other:
- sheet CM4_GPIO ( Ethernet, GPIO, SDCARD) ports: added 3V3, 5V, RXD4; removed +3.3v, +5v, TXD5
- sheet CM4_HighSpeed ports: added 3V3, 5V; removed +3.3v, +5v
- sheet Fan ports: added 12V, 3V3; removed +12v, +3.3v
- sheet PSUs ports: added 12V, 5V; removed +12v, +5v
- sheet USB2-HUB ports: added 3V3, 5V; removed +3.3v, +5v
Changed lines of the file:
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@@
     (effects (font (size 1.27 1.27)) (justify left bottom))
   )
-  (label "+5v" (at 104.14 125.73 0) (fields_autoplaced)
+  (label "5V" (at 104.14 125.73 0) (fields_autoplaced)
     (effects (font (size 1.27 1.27)) (justify left bottom))
   )
@@
     (effects (font (size 1.27 1.27)) (justify left bottom))
   )
-  (label "+12v" (at 67.945 88.9 0) (fields_autoplaced)
-    (effects (font (size 1.27 1.27)) (justify left bottom))
-  )
-  (label "+5v" (at 118.745 139.7 0) (fields_autoplaced)
+  (label "12V" (at 67.945 88.9 0) (fields_autoplaced)
+    (effects (font (size 1.27 1.27)) (justify left bottom))
+  )
+  (label "5V" (at 118.745 139.7 0) (fields_autoplaced)
     (effects (font (size 1.27 1.27)) (justify left bottom))
   )
@@
     (effects (font (size 1.27 1.27)) (justify left bottom))
   )
-  (label "+5v" (at 118.745 61.595 0) (fields_autoplaced)
+  (label "5V" (at 118.745 61.595 0) (fields_autoplaced)
     (effects (font (size 1.27 1.27)) (justify left bottom))
   )
@@
     (effects (font (size 1.27 1.27)) (justify left bottom))
   )
-  (label "+3.3v" (at 69.215 42.545 0) (fields_autoplaced)
+  (label "3V3" (at 69.215 42.545 0) (fields_autoplaced)
     (effects (font (size 1.27 1.27)) (justify left bottom))
   )
@@
     (effects (font (size 1.27 1.27)) (justify left bottom))
   )
-  (label "+12v" (at 104.14 121.92 0) (fields_autoplaced)
-    (effects (font (size 1.27 1.27)) (justify left bottom))
-  )
-  (label "+3.3v" (at 67.945 93.98 0) (fields_autoplaced)
-    (effects (font (size 1.27 1.27)) (justify left bottom))
-  )
-  (label "+3.3v" (at 118.745 142.24 0) (fields_autoplaced)
+  (label "12V" (at 104.14 121.92 0) (fields_autoplaced)
+    (effects (font (size 1.27 1.27)) (justify left bottom))
+  )
+  (label "3V3" (at 67.945 93.98 0) (fields_autoplaced)
+    (effects (font (size 1.27 1.27)) (justify left bottom))
+  )
+  (label "3V3" (at 118.745 142.24 0) (fields_autoplaced)
     (effects (font (size 1.27 1.27)) (justify left bottom))
   )
@@
     (effects (font (size 1.27 1.27)) (justify left bottom))
   )
-  (label "+5v" (at 69.215 36.195 0) (fields_autoplaced)
+  (label "5V" (at 69.215 36.195 0) (fields_autoplaced)
     (effects (font (size 1.27 1.27)) (justify left bottom))
   )
@@
     (effects (font (size 1.27 1.27)) (justify left bottom))
   )
-  (label "+3.3v" (at 118.745 65.405 0) (fields_autoplaced)
+  (label "3V3" (at 118.745 65.405 0) (fields_autoplaced)
     (effects (font (size 1.27 1.27)) (justify left bottom))
   )
@@
       (effects (font (size 1.27 1.27)) (justify right))
     )
-    (pin "+5v" input (at 127.635 139.7 180)
-      (effects (font (size 1.27 1.27)) (justify left))
-    )
-    (pin "+3.3v" output (at 127.635 142.24 180)
+    (pin "5V" input (at 127.635 139.7 180)
+      (effects (font (size 1.27 1.27)) (justify left))
+    )
+    (pin "3V3" output (at 127.635 142.24 180)
       (effects (font (size 1.27 1.27)) (justify left))
     )
@@
       (effects (font (size 1.27 1.27)) (justify right))
     )
-    (pin "TXD0" output (at 164.465 116.84 0)
-      (effects (font (size 1.27 1.27)) (justify right))
-    )
-    (pin "RXD0" input (at 164.465 114.3 0)
+    (pin "TXD0" output (at 164.465 139.7 0)
+      (effects (font (size 1.27 1.27)) (justify right))
+    )
+    (pin "RXD0" input (at 164.465 137.16 0)
       (effects (font (size 1.27 1.27)) (justify right))
     )
@@
       (effects (font (size 1.27 1.27)) (justify right))
     )
-    (pin "TXD5" output (at 164.465 137.16 0)
-      (effects (font (size 1.27 1.27)) (justify right))
-    )
-    (pin "TXD4" output (at 164.465 139.7 0)
-      (effects (font (size 1.27 1.27)) (justify right))
-    )
-    (pin "RST0" input (at 164.465 119.38 0)
+    (pin "RXD4" input (at 164.465 114.3 0)
+      (effects (font (size 1.27 1.27)) (justify right))
+    )
+    (pin "TXD4" output (at 164.465 116.84 0)
+      (effects (font (size 1.27 1.27)) (justify right))
+    )
+    (pin "RST0" output (at 164.465 142.24 0)
       (effects (font (size 1.27 1.27)) (justify right))
     )
@@
       (effects (font (size 1.27 1.27)) (justify right))
     )
-    (pin "RST4" input (at 164.465 142.24 0)
-      (effects (font (size 1.27 1.27)) (justify right))
-    )
-    (pin "PLUG4" input (at 164.465 134.62 0)
-      (effects (font (size 1.27 1.27)) (justify right))
-    )
-    (pin "RST3" input (at 164.465 130.81 0)
-      (effects (font (size 1.27 1.27)) (justify right))
-    )
-    (pin "PLUG0" input (at 164.465 111.76 0)
+    (pin "RST4" output (at 164.465 119.38 0)
+      (effects (font (size 1.27 1.27)) (justify right))
+    )
+    (pin "PLUG4" input (at 164.465 111.76 0)
+      (effects (font (size 1.27 1.27)) (justify right))
+    )
+    (pin "RST3" output (at 164.465 130.81 0)
+      (effects (font (size 1.27 1.27)) (justify right))
+    )
+    (pin "PLUG0" input (at 164.465 134.62 0)
       (effects (font (size 1.27 1.27)) (justify right))
     )
@@
       (effects (font (size 1.27 1.27)) (justify left))
     )
-    (pin "+5v" input (at 127.635 61.595 180)
-      (effects (font (size 1.27 1.27)) (justify left))
-    )
-    (pin "+3.3v" input (at 127.635 65.405 180)
+    (pin "5V" input (at 127.635 61.595 180)
+      (effects (font (size 1.27 1.27)) (justify left))
+    )
+    (pin "3V3" input (at 127.635 65.405 180)
       (effects (font (size 1.27 1.27)) (justify left))
     )
@@
       (effects (font (size 1.27 1.27)) (justify left top))
     )
-    (pin "+5v" output (at 101.6 125.73 0)
-      (effects (font (size 1.27 1.27)) (justify right))
-    )
-    (pin "+12v" output (at 101.6 121.92 0)
+    (pin "5V" output (at 101.6 125.73 0)
+      (effects (font (size 1.27 1.27)) (justify right))
+    )
+    (pin "12V" output (at 101.6 121.92 0)
       (effects (font (size 1.27 1.27)) (justify right))
     )
@@
       (effects (font (size 1.27 1.27)) (justify right))
     )
-    (pin "+5v" input (at 76.835 36.195 180)
-      (effects (font (size 1.27 1.27)) (justify left))
-    )
-    (pin "+3.3v" input (at 76.835 42.545 180)
+    (pin "5V" input (at 76.835 36.195 180)
+      (effects (font (size 1.27 1.27)) (justify left))
+    )
+    (pin "3V3" input (at 76.835 42.545 180)
       (effects (font (size 1.27 1.27)) (justify left))
     )
@@
       (effects (font (size 1.27 1.27)) (justify right))
     )
-    (pin "+3.3v" input (at 76.835 93.98 180)
+    (pin "3V3" input (at 76.835 93.98 180)
       (effects (font (size 1.27 1.27)) (justify left))
     )
@@
       (effects (font (size 1.27 1.27)) (justify right))
     )
-    (pin "+12v" input (at 76.835 88.9 180)
+    (pin "12V" input (at 76.835 88.9 180)
       (effects (font (size 1.27 1.27)) (justify left))
     )
@@
       (effects (font (size 1.27 1.27)) (justify left))
     )
-    (pin "PLUG0" input (at 182.245 111.76 180)
+    (pin "PLUG0" output (at 182.245 111.76 180)
       (effects (font (size 1.27 1.27)) (justify left))
     )
@@
       (effects (font (size 1.27 1.27)) (justify left))
     )
-    (pin "RXD1" input (at 182.245 125.73 180)
+    (pin "RXD1" output (at 182.245 125.73 180)
       (effects (font (size 1.27 1.27)) (justify left))
     )
@@
       (effects (font (size 1.27 1.27)) (justify left))
     )
-    (pin "PLUG2" input (at 182.245 134.62 180)
+    (pin "PLUG2" output (at 182.245 134.62 180)
       (effects (font (size 1.27 1.27)) (justify left))
     )
@@
       (effects (font (size 1.27 1.27)) (justify left))
     )
-    (pin "PLUG1" input (at 182.245 123.19 180)
+    (pin "PLUG1" output (at 182.245 123.19 180)
       (effects (font (size 1.27 1.27)) (justify left))
     )
@@
       (effects (font (size 1.27 1.27)) (justify left))
     )
-    (pin "SCL" input (at 182.245 104.775 180)
+    (pin "SCL" bidirectional (at 182.245 104.775 180)
       (effects (font (size 1.27 1.27)) (justify left))
     )
@@
       (effects (font (size 1.27 1.27)) (justify left))
     )
-    (pin "RXD2" input (at 182.245 137.16 180)
-      (effects (font (size 1.27 1.27)) (justify left))
-    )
-    (pin "RXD0" input (at 182.245 114.3 180)
-      (effects (font (size 1.27 1.27)) (justify left))
-    )
+    (pin "RXD2" output (at 182.245 137.16 180)
+      (effects (font (size 1.27 1.27)) (justify left))
+    )
+    (pin "RXD0" output (at 182.245 114.3 180)
+      (effects (font (size 1.27 1.27)) (justify left))
+    )
