File: hashboards.kicad_sch (KiCad schematic)
At the start: 22 parts, among them J13 Hashboard0, J14 Hashboard1, J15 Hashboard2, U10 PCA9546ARGVR

Commit message: added more USB ports.. placing
Parts:
- removed J13: Hashboard0, bitcart:CONN-TH_X2026WV-2-09D-46SN, symbol Connector_Generic:Conn_02x09_Odd_Even
- removed J14: Hashboard1, bitcart:CONN-TH_X2026WV-2-09D-46SN, symbol Connector_Generic:Conn_02x09_Odd_Even
- removed J15: Hashboard2, bitcart:CONN-TH_X2026WV-2-09D-46SN, symbol Connector_Generic:Conn_02x09_Odd_Even
- removed R28, R29, R30, R31, R32, R33, R34, R35, R36, R37, R38, R39, R40, R41, R42, R43, R44, R45: 4.7K, Resistor_SMD:R_0805_2012Metric, symbol Device:R_US
- removed U10: PCA9546ARGVR, bitcart:QFN-16_EP_4x4_Pitch0.65mm, symbol bitcart:PCA9546ARGVR
Connections:
- no-connect marks 6 -> 0
